File: msisdr.kicad_pcb (KiCad board)
At the start: 2 copper layers, 46.3 x 90.7 mm, 70 parts, among them J1 VCC_GPIO, J10 SMA_VHF1, J11 USB_OTG, J2 GPIO0, J3 GPIO1, J4 GPIO2, J5 GPIO3, J6 SMA_0_30MHZ, J7 SMA_30_60MHZ, J8 SMA_VHF2, J9 SMA_UHF, U1 msi2500, U2 msi001, U3 LP5900SDX-2.8, U4 AP7313-30SAG, Y1 24MHz

Commit message: adjust some line and hole
Parts:
- moved REF** 1.50 mm to (154.5, 124.0)
- moved REF** 1.50 mm to (118.0, 124.0)
- moved REF** 1.50 mm to (154.5, 50.0)
- moved REF** 1.50 mm to (118.0, 50.0)
Routing:
- net VHF_120_250MHZ: track 31.4 -> 32.6 mm
Changed lines of the file:
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@@
     (thickness 1.6)
     (drawings 5)
-    (tracks 817)
+    (tracks 823)
     (zones 0)
     (modules 70)
@@
     (mod_text_size 1 1)
     (mod_text_width 0.15)
-    (pad_size 1.524 1.524)
-    (pad_drill 0.762)
+    (pad_size 4.064 4.064)
+    (pad_drill 3)
     (pad_to_mask_clearance 0.2)
     (aux_axis_origin 0 0)
@@
   )
   (module Connectors:1pin (layer F.Cu)
-    (at 156 124)
+    (at 154.5 124)
     (descr "module 1 pin (ou trou mecanique de percage)")
     (tags DEV)
@@
   )
   (module Connectors:1pin (layer F.Cu)
-    (at 116.5 124)
+    (at 118 124)
     (descr "module 1 pin (ou trou mecanique de percage)")
     (tags DEV)
@@
   )
   (module Connectors:1pin (layer F.Cu)
-    (at 156 50)
+    (at 154.5 50)
     (descr "module 1 pin (ou trou mecanique de percage)")
     (tags DEV)
@@
   )
   (module Connectors:1pin (layer F.Cu)
-    (at 116.5 50)
+    (at 118 50)
     (descr "module 1 pin (ou trou mecanique de percage)")
     (tags DEV)
@@
   (segment (start 128.039 102.166) (end 128.039 81.426) (width 0.2) (layer F.Cu) (net 25))
   (segment (start 130.549 104.676) (end 128.039 102.166) (width 0.2) (layer F.Cu) (net 25))
-  (segment (start 134.109 108.426) (end 134.109 109.35762) (width 0.2) (layer F.Cu) (net 26))
-  (segment (start 120.2055 124.3203) (end 120.2055 132.0692) (width 0.2) (layer F.Cu) (net 26))
-  (segment (start 120.21312 124.31268) (end 120.2055 124.3203) (width 0.2) (layer F.Cu) (net 26))
-  (via (at 120.21312 124.31268) (size 0.6) (drill 0.4) (layers F.Cu B.Cu) (net 26))
-  (segment (start 126.70536 117.82044) (end 120.21312 124.31268) (width 0.2) (layer B.Cu) (net 26))
-  (segment (start 130.08864 117.82044) (end 126.70536 117.82044) (width 0.2) (layer B.Cu) (net 26))
-  (segment (start 133.07568 114.8334) (end 130.08864 117.82044) (width 0.2) (layer B.Cu) (net 26))
-  (segment (start 133.07568 111.0234) (end 133.07568 114.8334) (width 0.2) (layer B.Cu) (net 26))
-  (segment (start 133.0452 110.99292) (end 133.07568 111.0234) (width 0.2) (layer B.Cu) (net 26))
-  (via (at 133.0452 110.99292) (size 0.6) (drill 0.4) (layers F.Cu B.Cu) (net 26))
-  (segment (start 133.14426 110.89386) (end 133.0452 110.99292) (width 0.2) (layer F.Cu) (net 26))
-  (segment (start 133.14426 110.32236) (end 133.14426 110.89386) (width 0.2) (layer F.Cu) (net 26))
+  (segment (start 121.3755 128.0392) (end 121.3608 128.0392) (width 0.2) (layer F.Cu) (net 26))
   (segment (start 134.109 109.35762) (end 133.14426 110.32236) (width 0.2) (layer F.Cu) (net 26))
+  (segment (start 133.14426 110.32236) (end 133.14426 110.89386) (width 0.2) (layer F.Cu) (net 26))
+  (segment (start 133.14426 110.89386) (end 133.0452 110.99292) (width 0.2) (layer F.Cu) (net 26))
+  (via (at 133.0452 110.99292) (size 0.6) (drill 0.4) (layers F.Cu B.Cu) (net 26))
+  (segment (start 133.0452 110.99292) (end 133.07568 111.0234) (width 0.2) (layer B.Cu) (net 26))
+  (segment (start 133.07568 111.0234) (end 133.07568 114.8334) (width 0.2) (layer B.Cu) (net 26))
+  (segment (start 133.07568 114.8334) (end 130.08864 117.82044) (width 0.2) (layer B.Cu) (net 26))
+  (segment (start 130.08864 117.82044) (end 126.70536 117.82044) (width 0.2) (layer B.Cu) (net 26))
+  (segment (start 126.70536 117.82044) (end 121.38312 120.28268) (width 0.2) (layer B.Cu) (net 26))
+  (via (at 121.38312 120.28268) (size 0.6) (drill 0.4) (layers F.Cu B.Cu) (net 26))
+  (segment (start 121.38312 120.28268) (end 121.3755 120.2903) (width 0.2) (layer F.Cu) (net 26))
+  (segment (start 121.3755 120.2903) (end 121.3755 128.0392) (width 0.2) (layer F.Cu) (net 26))
+  (segment (start 134.109 108.426) (end 134.109 109.35762) (width 0.2) (layer F.Cu) (net 26))
+  (segment (start 120.2055 129.1945) (end 120.2055 132.0692) (width 0.2) (layer F.Cu) (net 26) (status 800000))
+  (segment (start 121.3608 128.0392) (end 120.2055 129.1945) (width 0.2) (layer F.Cu) (net 26))
   (segment (start 135.08736 110.61192) (end 135.08736 110.4646) (width 0.2) (layer F.Cu) (net 27))
   (segment (start 136.88568 131.88632) (end 136.88568 127.56388) (width 0.2) (layer F.Cu) (net 27))
@@
   (segment (start 135.08736 110.4646) (end 135.609 109.94296) (width 0.2) (layer F.Cu) (net 27))
   (segment (start 136.88568 131.88632) (end 136.7028 132.0692) (width 0.2) (layer F.Cu) (net 27))
-  (segment (start 137.609 108.426) (end 137.609 108.82064) (width 0.2) (layer F.Cu) (net 28))
-  (segment (start 152.5397 127.41402) (end 152.5397 132.12254) (width 0.2) (layer F.Cu) (net 28))
-  (segment (start 152.34412 127.21844) (end 152.5397 127.41402) (width 0.2) (layer F.Cu) (net 28))
-  (via (at 152.34412 127.21844) (size 0.6) (drill 0.4) (layers F.Cu B.Cu) (net 28))
-  (segment (start 152.34412 122.09272) (end 152.34412 127.21844) (width 0.2) (layer B.Cu) (net 28))
-  (segment (start 146.3802 116.1288) (end 152.34412 122.09272) (width 0.2) (layer B.Cu) (net 28))
-  (segment (start 146.3802 111.7092) (end 146.3802 116.1288) (width 0.2) (layer B.Cu) (net 28))
-  (segment (start 143.71066 109.03966) (end 146.3802 111.7092) (width 0.2) (layer B.Cu) (net 28))
-  (segment (start 140.31722 109.03966) (end 143.71066 109.03966) (width 0.2) (layer B.Cu) (net 28))
-  (segment (start 140.31468 109.0422) (end 140.31722 109.03966) (width 0.2) (layer B.Cu) (net 28))
-  (via (at 140.31468 109.0422) (size 0.6) (drill 0.4) (layers F.Cu B.Cu) (net 28))
-  (segment (start 137.83056 109.0422) (end 140.31468 109.0422) (width 0.2) (layer F.Cu) (net 28))
+  (segment (start 152.5397 132.12254) (end 152.5397 129.0297) (width 0.2) (layer F.Cu) (net 28) (status 400000))
   (segment (start 137.609 108.82064) (end 137.83056 109.0422) (width 0.2) (layer F.Cu) (net 28))
+  (segment (start 137.83056 109.0422) (end 140.31468 109.0422) (width 0.2) (layer F.Cu) (net 28))
+  (via (at 140.31468 109.0422) (size 0.6) (drill 0.4) (layers F.Cu B.Cu) (net 28))
+  (segment (start 140.31468 109.0422) (end 140.31722 109.03966) (width 0.2) (layer B.Cu) (net 28))
+  (segment (start 140.31722 109.03966) (end 143.71066 109.03966) (width 0.2) (layer B.Cu) (net 28))
+  (segment (start 143.71066 109.03966) (end 146.3802 111.7092) (width 0.2) (layer B.Cu) (net 28))
+  (segment (start 146.3802 111.7092) (end 146.3802 116.1288) (width 0.2) (layer B.Cu) (net 28))
+  (segment (start 146.3802 116.1288) (end 150.66412 121.47272) (width 0.2) (layer B.Cu) (net 28))
+  (segment (start 150.66412 121.47272) (end 150.66412 126.59844) (width 0.2) (layer B.Cu) (net 28))
+  (via (at 150.66412 126.59844) (size 0.6) (drill 0.4) (layers F.Cu B.Cu) (net 28))
+  (segment (start 137.609 108.82064) (end 137.609 108.426) (width 0.2) (layer F.Cu) (net 28))
+  (segment (start 150.66412 127.77412) (end 150.66412 126.59844) (width 0.2) (layer F.Cu) (net 28))
+  (segment (start 151.11 128.22) (end 150.66412 127.77412) (width 0.2) (layer F.Cu) (net 28))
+  (segment (start 151.73 128.22) (end 151.11 128.22) (width 0.2) (layer F.Cu) (net 28))
+  (segment (start 152.5397 129.0297) (end 151.73 128.22) (width 0.2) (layer F.Cu) (net 28))
   (segment (start 126.7968 123.2129) (end 128.81098 123.2129) (width 0.2) (layer F.Cu) (net 34))
   (segment (start 130.1376 120.54516) (end 131.10972 120.54516) (width 0.2) (layer F.Cu) (net 34))
@@
   (segment (start 126.7968 121.3129) (end 123.44392 121.3129) (width 0.2) (layer F.Cu) (net 58))
   (segment (start 123.44392 121.3129) (end 123.03506 120.90404) (width 0.2) (layer F.Cu) (net 58))
-  (segment (start 131.569 45.396) (end 140.469 45.396) (width 0.2) (layer F.Cu) (net 60) (status C00000))
-  (segment (start 140.469 45.396) (end 140.469 50.896) (width 0.2) (layer F.Cu) (net 60) (status C00000))
-  (segment (start 131.569 45.396) (end 131.569 50.896) (width 0.2) (layer F.Cu) (net 60) (status C00000))
+  (segment (start 131.569 45.396) (end 140.469 45.396) (width 0.2) (layer F.Cu) (net 60))
+  (segment (start 140.469 45.396) (end 140.469 50.896) (width 0.2) (layer F.Cu) (net 60))
+  (segment (start 131.569 45.396) (end 131.569 50.896) (width 0.2) (layer F.Cu) (net 60))
   (segment (start 149.919 65.626) (end 150.59916 65.626) (width 0.2) (layer F.Cu) (net 61))
   (segment (start 151.01316 62.6364) (end 149.1086 62.6364) (width 0.2) (layer F.Cu) (net 61))

Commit message: finally version of pcb
Routing:
- added copper zone on B.Cu, net GND
- added copper zone on F.Cu, net GND
Changed lines of the file:
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@@
   (general
     (links 234)
-    (no_connects 2)
-    (area 113.056599 42.470999 159.490481 144.007101)
+    (no_connects 0)
+    (area 99.214908 36.92012 159.490481 144.007101)
     (thickness 1.6)
-    (drawings 5)
+    (drawings 7)
     (tracks 823)
     (zones 0)
@@
   (layers
     (0 F.Cu signal)
-    (31 B.Cu signal)
+    (31 B.Cu signal hide)
     (32 B.Adhes user)
     (33 F.Adhes user)
@@
     (visible_elements 7FFEFFFF)
     (pcbplotparams
-      (layerselection 0x00030_80000001)
+      (layerselection 0x01fff_80000001)
       (usegerberextensions false)
       (excludeedgelayer true)
@@
       (outputformat 1)
       (mirror false)
-      (drillshape 1)
+      (drillshape 0)
       (scaleselection 1)
-      (outputdirectory ""))
+      (outputdirectory Gerber/))
   )
   (net 0 "")
@@
     )
   )
+  (dimension 90.600001 (width 0.3) (layer Eco2.User)
+    (gr_text "90.600 mm" (at 105.714907 88.809181 89.99367596) (layer Eco2.User)
+      (effects (font (size 1.5 1.5) (thickness 0.3)))
+    )
+    (feature1 (pts (xy 113.13 134.11) (xy 104.359907 134.109032)))
+    (feature2 (pts (xy 113.14 43.51) (xy 104.369907 43.509032)))
+    (crossbar (pts (xy 107.069907 43.50933) (xy 107.059907 134.10933)))
+    (arrow1a (pts (xy 107.059907 134.10933) (xy 106.473611 132.982762)))
+    (arrow1b (pts (xy 107.059907 134.10933) (xy 107.646452 132.982891)))
+    (arrow2a (pts (xy 107.069907 43.50933) (xy 106.483362 44.635769)))
+    (arrow2b (pts (xy 107.069907 43.50933) (xy 107.656203 44.635898)))
+  )
+  (dimension 46.27001 (width 0.3) (layer Eco2.User)
+    (gr_text "46.270 mm" (at 136.268378 38.285119 359.9628512) (layer Eco2.User)
+      (effects (font (size 1.5 1.5) (thickness 0.3)))
+    )
+    (feature1 (pts (xy 159.4 43.51) (xy 159.404254 36.95012)))
+    (feature2 (pts (xy 113.13 43.48) (xy 113.134254 36.92012)))
+    (crossbar (pts (xy 113.132503 39.620119) (xy 159.402503 39.650119)))
+    (arrow1a (pts (xy 159.402503 39.650119) (xy 158.275619 40.235809)))
+    (arrow1b (pts (xy 159.402503 39.650119) (xy 158.27638 39.062968)))
+    (arrow2a (pts (xy 113.132503 39.620119) (xy 114.258626 40.20727)))
+    (arrow2b (pts (xy 113.132503 39.620119) (xy 114.259387 39.034429)))
+  )
   (gr_line (start 159.41548 134.13232) (end 113.13668 134.13232) (angle 90) (layer Edge.Cuts) (width 0.15))
   (gr_line (start 113.1316 134.08914) (end 113.157 134.08914) (angle 90) (layer Edge.Cuts) (width 0.15))
@@
   (segment (start 121.3755 120.2903) (end 121.3755 128.0392) (width 0.2) (layer F.Cu) (net 26))
   (segment (start 134.109 108.426) (end 134.109 109.35762) (width 0.2) (layer F.Cu) (net 26))
-  (segment (start 120.2055 129.1945) (end 120.2055 132.0692) (width 0.2) (layer F.Cu) (net 26) (status 800000))
+  (segment (start 120.2055 129.1945) (end 120.2055 132.0692) (width 0.2) (layer F.Cu) (net 26))
   (segment (start 121.3608 128.0392) (end 120.2055 129.1945) (width 0.2) (layer F.Cu) (net 26))
   (segment (start 135.08736 110.61192) (end 135.08736 110.4646) (width 0.2) (layer F.Cu) (net 27))
@@
   (segment (start 135.08736 110.4646) (end 135.609 109.94296) (width 0.2) (layer F.Cu) (net 27))
   (segment (start 136.88568 131.88632) (end 136.7028 132.0692) (width 0.2) (layer F.Cu) (net 27))
-  (segment (start 152.5397 132.12254) (end 152.5397 129.0297) (width 0.2) (layer F.Cu) (net 28) (status 400000))
+  (segment (start 152.5397 132.12254) (end 152.5397 129.0297) (width 0.2) (layer F.Cu) (net 28))
   (segment (start 137.609 108.82064) (end 137.83056 109.0422) (width 0.2) (layer F.Cu) (net 28))
   (segment (start 137.83056 109.0422) (end 140.31468 109.0422) (width 0.2) (layer F.Cu) (net 28))
@@
   (segment (start 138.909 52.95) (end 146.959 52.95) (width 0.2) (layer F.Cu) (net 61))
   (segment (start 137.619 52.436) (end 138.909 52.95) (width 0.2) (layer F.Cu) (net 61))
+  (zone (net 35) (net_name GND) (layer F.Cu) (hatch edge 0.508)
+    (connect_pads (clearance 0.508))
+    (min_thickness 0.254)
+    (fill yes (arc_segments 16) (thermal_gap 0.508) (thermal_bridge_width 0.508))
+    (polygon
+      (pts
+        (xy 113.15 43.48) (xy 159.39 43.5) (xy 159.43 134.13) (xy 113.15 134.1)
+      )
+    )
+  )
+  (zone (net 35) (net_name GND) (layer B.Cu) (hatch edge 0.508)
+    (connect_pads (clearance 0.508))
+    (min_thickness 0.254)
+    (fill yes (arc_segments 16) (thermal_gap 0.508) (thermal_bridge_width 0.508))
+    (polygon
+      (pts
+        (xy 159.4 134.13) (xy 113.16 134.14) (xy 113.14 43.51) (xy 159.38 43.46)
+      )
+    )
+  )
 )
