File: rf_parts.sch (KiCad schematic (older format))
At the start: 19 parts

Commit message: msi2500 full pcb design
Parts:
- removed C?: 100nF, symbol C
- removed C?: 2.7pF, symbol C
- removed C?: 82pF, symbol C
- removed C?: 180pF, symbol C
- removed J?: SMA_0_12MHZ, symbol Conn_01x02
- removed J?: SMA_12_30MHZ, symbol Conn_01x02
- removed J?: SMA_30_60MHZ, symbol Conn_01x02
- removed J? (x3): Conn_01x02, symbol Conn_01x02
- removed L?: 330nH, symbol L
- removed L?: 470nH, symbol L
- added C27: 1nF, Capacitors_SMD:C_0603, symbol C
- added C28, C31: 160pF, Capacitors_SMD:C_0603, symbol C
- added C32: 56pF, Capacitors_SMD:C_0603, symbol C
- added J2: SMA_0_30MHZ, sma:SMA_OPL_EM, symbol Conn_01x03
- added J3: SMA_30_60MHZ, sma:SMA_OPL_EM, symbol Conn_01x03
- added J4: SMA_VHF2, sma:SMA_OPL_EMPTYHEAD, symbol Conn_01x03
- added J5: SMA_UHF, sma:SMA_OPL_EMPTYHEAD, symbol Conn_01x03
- added J6: SMA_VHF1, sma:SMA_OPL_EMPTYHEAD, symbol Conn_01x03
- added L2: 270nH, Inductors_SMD:L_0805, symbol L
- added L4: 150nH, Inductors_SMD:L_0805, symbol L
- added L6: 330nH, Inductors_SMD:L_0805, symbol L
- C26: renamed from C?; value 3.3pF -> 470nF; footprint (none) -> Capacitors_SMD:C_0805
- C29, C33: renamed from C?; footprint (none) -> Capacitors_SMD:C_0603
- C30: renamed from C?; value 120pF -> 56pF; footprint (none) -> Capacitors_SMD:C_0603
- L1, L5: renamed from L?; footprint (none) -> Inductors_SMD:L_0805
- L3: renamed from L?; value 1000nH -> 330nH; footprint (none) -> Inductors_SMD:L_0805
Connections:
- wire segments 44 -> 53
Other:
- moved on the sheet: C26, C29, C30, C33, L1, L3, L5

Commit message: update and fix bug
Parts:
- renumbered C26 to C27, C27 to C28, C30 to C29, C29 to C30, C28 to C31, C33 to C32, C31 to C33, C32 to C34, J6 to J10, J2 to J6, J3 to J7, J4 to J8, J5 to J9, L5 to L2, L2 to L4, L4 to L5
Changed lines of the file:
@@
 $EndComp
 $Comp
-L C C26
+L C C27
 U 1 1 5C6942E9
 P 3250 2500
-F 0 "C26" H 3275 2600 50  0000 L CNN
+F 0 "C27" H 3275 2600 50  0000 L CNN
 F 1 "470nF" H 3275 2400 50  0000 L CNN
 F 2 "Capacitors_SMD:C_0805" H 3288 2350 50  0001 C CNN
@@
 $EndComp
 $Comp
-L C C30
+L C C29
 U 1 1 5C694335
 P 3750 3200
-F 0 "C30" H 3775 3300 50  0000 L CNN
+F 0 "C29" H 3775 3300 50  0000 L CNN
 F 1 "56pF" H 3775 3100 50  0000 L CNN
 F 2 "Capacitors_SMD:C_0603" H 3788 3050 50  0001 C CNN
@@
 $EndComp
 $Comp
-L C C29
+L C C30
 U 1 1 5C694F53
 P 3850 4250
-F 0 "C29" H 3875 4350 50  0000 L CNN
+F 0 "C30" H 3875 4350 50  0000 L CNN
 F 1 "3.9pF" H 3875 4150 50  0000 L CNN
 F 2 "Capacitors_SMD:C_0603" H 3888 4100 50  0001 C CNN
@@
 $EndComp
 $Comp
-L L L5
+L L L2
 U 1 1 5C694FBF
 P 3850 4650
-F 0 "L5" V 3800 4650 50  0000 C CNN
+F 0 "L2" V 3800 4650 50  0000 C CNN
 F 1 "330nH" V 3925 4650 50  0000 C CNN
 F 2 "Inductors_SMD:L_0805" H 3850 4650 50  0001 C CNN
@@
 $EndComp
 $Comp
-L C C33
+L C C32
 U 1 1 5C69501A
 P 4900 4400
-F 0 "C33" H 4925 4500 50  0000 L CNN
+F 0 "C32" H 4925 4500 50  0000 L CNN
 F 1 "39pF" H 4925 4300 50  0000 L CNN
 F 2 "Capacitors_SMD:C_0603" H 4938 4250 50  0001 C CNN
@@
 Wire Wire Line
 	6300 4400 5050 4400
-Text GLabel 9050 2700 2    20   Output ~ 0
+Text GLabel 9050 2700 2    20   Input ~ 0
 VHF_120_250MHZ
-Text GLabel 9050 3450 2    20   Output ~ 0
+Text GLabel 9050 3450 2    20   Input ~ 0
 UHF_400_1000MHZ
-Text GLabel 8900 4200 2    20   Output ~ 0
+Text GLabel 8900 4200 2    20   Input ~ 0
 VHF_50_120MHZ
 $Comp
@@
 Wire Wire Line
 	8350 4200 8900 4200
-Text GLabel 6500 3600 2    20   Output ~ 0
+Text GLabel 6500 3600 2    20   Input ~ 0
 HFPORT
 $Comp
-L C C27
+L C C28
 U 1 1 5C694529
 P 3250 2950
-F 0 "C27" H 3275 3050 50  0000 L CNN
+F 0 "C28" H 3275 3050 50  0000 L CNN
 F 1 "1nF" H 3275 2850 50  0000 L CNN
 F 2 "Capacitors_SMD:C_0603" H 3288 2800 50  0001 C CNN
@@
 $EndComp
 $Comp
-L L L2
+L L L4
 U 1 1 5C6947E7
 P 4450 2500
-F 0 "L2" V 4400 2500 50  0000 C CNN
+F 0 "L4" V 4400 2500 50  0000 C CNN
 F 1 "270nH" V 4525 2500 50  0000 C CNN
 F 2 "Inductors_SMD:L_0805" H 4450 2500 50  0001 C CNN
@@
 $EndComp
 $Comp
-L L L4
+L L L5
 U 1 1 5C694859
 P 4900 2500
-F 0 "L4" V 4850 2500 50  0000 C CNN
+F 0 "L5" V 4850 2500 50  0000 C CNN
 F 1 "150nH" V 4975 2500 50  0000 C CNN
 F 2 "Inductors_SMD:L_0805" H 4900 2500 50  0001 C CNN
@@
 $EndComp
 $Comp
-L C C28
+L C C31
 U 1 1 5C694ABC
 P 4250 3200
-F 0 "C28" H 4275 3300 50  0000 L CNN
+F 0 "C31" H 4275 3300 50  0000 L CNN
 F 1 "160pF" H 4275 3100 50  0000 L CNN
 F 2 "Capacitors_SMD:C_0603" H 4288 3050 50  0001 C CNN
@@
 $EndComp
 $Comp
-L C C31
+L C C33
 U 1 1 5C694B0D
 P 5150 3200
-F 0 "C31" H 5175 3300 50  0000 L CNN
+F 0 "C33" H 5175 3300 50  0000 L CNN
 F 1 "160pF" H 5175 3100 50  0000 L CNN
 F 2 "Capacitors_SMD:C_0603" H 5188 3050 50  0001 C CNN
@@
 $EndComp
 $Comp
-L C C32
+L C C34
 U 1 1 5C694B60
 P 5750 3200
-F 0 "C32" H 5775 3300 50  0000 L CNN
+F 0 "C34" H 5775 3300 50  0000 L CNN
 F 1 "56pF" H 5775 3100 50  0000 L CNN
 F 2 "Capacitors_SMD:C_0603" H 5788 3050 50  0001 C CNN
@@
 Connection ~ 6300 3600
 $Comp
-L Conn_01x03 J2
+L Conn_01x03 J6
 U 1 1 5C696A99
 P 1800 2600
-F 0 "J2" H 1800 2800 50  0000 C CNN
+F 0 "J6" H 1800 2800 50  0000 C CNN
 F 1 "SMA_0_30MHZ" H 1800 2400 50  0000 C CNN
 F 2 "sma:SMA_OPL_EM" H 1800 2600 50  0001 C CNN
@@
 Connection ~ 2150 2600
 $Comp
-L Conn_01x03 J3
+L Conn_01x03 J7
 U 1 1 5C696D80
 P 1900 4350
-F 0 "J3" H 1900 4550 50  0000 C CNN
+F 0 "J7" H 1900 4550 50  0000 C CNN
 F 1 "SMA_30_60MHZ" H 1900 4150 50  0000 C CNN
 F 2 "sma:SMA_OPL_EM" H 1900 4350 50  0001 C CNN
@@
 Connection ~ 2200 4350
 $Comp
-L Conn_01x03 J4
+L Conn_01x03 J8
 U 1 1 5C69724D
 P 8150 2800
-F 0 "J4" H 8150 3000 50  0000 C CNN
+F 0 "J8" H 8150 3000 50  0000 C CNN
 F 1 "SMA_VHF2" H 8150 2600 50  0000 C CNN
 F 2 "sma:SMA_OPL_EMPTYHEAD" H 8150 2800 50  0001 C CNN
@@
 $EndComp
 $Comp
-L Conn_01x03 J5
+L Conn_01x03 J9
 U 1 1 5C6972AA
 P 8150 3550
-F 0 "J5" H 8150 3750 50  0000 C CNN
+F 0 "J9" H 8150 3750 50  0000 C CNN
 F 1 "SMA_UHF" H 8150 3350 50  0000 C CNN
 F 2 "sma:SMA_OPL_EMPTYHEAD" H 8150 3550 50  0001 C CNN
@@
 $EndComp
 $Comp
-L Conn_01x03 J6
+L Conn_01x03 J10
 U 1 1 5C697362
 P 8150 4300
-F 0 "J6" H 8150 4500 50  0000 C CNN
+F 0 "J10" H 8150 4500 50  0000 C CNN
 F 1 "SMA_VHF1" H 8150 4100 50  0000 C CNN
 F 2 "sma:SMA_OPL_EMPTYHEAD" H 8150 4300 50  0001 C CNN
